File: test_temp/untitled.brd (EAGLE design)
At the start: 88.9 x 50.8 mm, 14 parts, among them IC1 74ABT125PW, U1 DS31126, U2 DS31126, U3 DS31126

Commit message: sent to fab + parts on order
if this works ill be surprised. it should... but man, I see alot is issues. *fingers crossed*
Parts:
- removed U1: DS31126, ds31126:SOT23
- added IC2: 74ABT125PW, 74xx-eu:TSSOP14
- IC1: value 74ABT125PW -> DS31126; device 74xx-us:TSSOP14 -> ds31126:SOT23
- R2: value 10k -> 18; device rcl:R0603 -> rcl:R2512W
- R5: value 18 -> 10k; device rcl:R2512W -> rcl:R0603
- moved R2 25.7 mm to (20.6, 45.5), turned to 90 degrees
- moved R4 16.3 mm to (20.6, 29.2)
- moved IC1 14.2 mm to (22.1, 39.4), turned to 90 degrees
- moved R5 13.8 mm to (19.3, 15.5), turned to 180 degrees
- moved R3 5.01 mm to (21.8, 19.8), turned to 0 degrees
- renumbered U$1 to NICR1, U2 to IC3, U3 to IC4
Connections:
- removed net EN1: IC1.1, SV1.3
- removed net EN2: IC1.4, SV1.4
- removed net EN3: IC1.10, SV1.5
- new net !EN1: IC2.1, SV1.3
- new net !EN2: IC2.4, SV1.4
- new net !EN3: IC2.10, SV1.6
- new net PWM_IN: IC2.12, SV1.5
- net E1: now also R2.2; no longer R4.2
- net E1_EN: now also IC1.G, IC2.3; no longer IC1.3, U1.G
- net E2: now also R4.2; no longer R5.2
- net E2_EN: now also IC2.6, R3.2; no longer IC1.6, R2.2
- net E3_EN: now also IC2.8, R5.2; no longer IC1.8, R3.2
- net GND: now also IC1.S, IC2.13, IC2.7, R5.1; no longer IC1.7, R2.1, U1.S
- net N$1: now also IC1.D, R2.1; no longer R4.1, U1.D
- net N$2: now also R4.1; no longer R5.1
- net PWM: now also IC2.11, IC2.2, IC2.5, IC2.9; no longer IC1.2, IC1.5, IC1.9, SV1.6
- net VCC: now also IC2.14; no longer IC1.14
Routing:
- net EN1: track 50.8 -> 0.00 mm, vias 2 -> 0
- net EN2: track 48.7 -> 0.00 mm, vias 2 -> 0
- net !EN1: track 0.00 -> 48.1 mm, vias 0 -> 1
- net !EN2: track 0.00 -> 44.7 mm, vias 0 -> 1
- net PWM_IN: track 0.00 -> 36.6 mm
- net EN3: track 36.3 -> 0.00 mm
- net !EN3: track 0.00 -> 33.5 mm
- net PWM: track 43.4 -> 13.4 mm
Other:
- board text added: "!EN1"
- board text added: "!EN2"
- board text added: "!EN3"
- board text added: "2021"
- board text added: "36AWG NiCr may open at high current Sink .6A@12v - .5A@9v - .2A@5v"
- board text added: "Drag Durring Activation"
- board text added: "PWM"
- board text added: "VCC"
- board text added: "WARNING PCB May Fail"
- board text added: "reserved for future use"
- board text removed: "EN1"
- board text removed: "EN2"
- board text removed: "EN3"
- board text removed: "PWM 5K"
- board text removed: "R4-R5-R6 may get warm"
- board text removed: "Vcc"

Commit message: fixed sch
Parts:
- IC1, IC3, IC4: value DS31126 -> DMN3150L-7
Changed lines of the file:
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@@
 <drawing>
 <settings>
-<setting alwaysvectorfont="yes"/>
+<setting alwaysvectorfont="no"/>
 <setting verticaltext="up"/>
 </settings>
@@
 <elements>
 <element name="NICR1" library="logo_wire" package="LAYOUT_A" value="HOT_WIRE" x="3.175" y="30.48" smashed="yes"/>
-<element name="IC1" library="ds31126" package="SOT23" value="DS31126" x="22.098" y="39.37" smashed="yes" rot="R90">
+<element name="IC1" library="ds31126" package="SOT23" value="DMN3150L-7" x="22.098" y="39.37" smashed="yes" rot="R90">
 <attribute name="NAME" x="25.273" y="38.989" size="0.8128" layer="25" font="vector" ratio="15" rot="R90"/>
 </element>
-<element name="IC3" library="ds31126" package="SOT23" value="DS31126" x="21.59" y="23.114" smashed="yes" rot="R90">
+<element name="IC3" library="ds31126" package="SOT23" value="DMN3150L-7" x="21.59" y="23.114" smashed="yes" rot="R90">
 <attribute name="NAME" x="24.765" y="22.479" size="0.8128" layer="25" font="vector" ratio="15" rot="R90"/>
 </element>
-<element name="IC4" library="ds31126" package="SOT23" value="DS31126" x="19.304" y="11.938" smashed="yes" rot="R270">
+<element name="IC4" library="ds31126" package="SOT23" value="DMN3150L-7" x="19.304" y="11.938" smashed="yes" rot="R270">
 <attribute name="NAME" x="21.971" y="12.573" size="0.8128" layer="25" font="vector" ratio="15" rot="R270"/>
 </element>
