File: test_temp/untitled.sch (EAGLE design)
At the start: 14 parts, among them IC1 74ABT125PW, U1 DS31126, U2 DS31126, U3 DS31126

Commit message: sent to fab + parts on order
if this works ill be surprised. it should... but man, I see alot is issues. *fingers crossed*
Parts:
- removed U1: DS31126, ds31126:DS31126
- added IC2: 74ABT125PW, 74xx-eu:74ABT125PW
- IC1: value 74ABT125PW -> DS31126; device 74xx-us:74ABT125PW -> ds31126:DS31126
- R2: value 10k -> 18; device rcl:R-US_R0603 -> rcl:R-US_R2512W
- R5: value 18 -> 10k; device rcl:R-US_R2512W -> rcl:R-US_R0603
- renumbered U$1 to NICR1, U2 to IC3, U3 to IC4
Connections:
- removed net EN1: IC1A.OE, SV1.3
- removed net EN2: IC1B.OE, SV1.4
- removed net EN3: IC1C.OE, SV1.5
- new net !EN1: IC2A.OE, SV1.3
- new net !EN2: IC2B.OE, SV1.4
- new net !EN3: IC2C.OE, SV1.6
- new net PWM_IN: IC2D.I, SV1.5
- net E1: now also R2.2; no longer R4.2
- net E1_EN: now also IC1.G, IC2A.O; no longer IC1A.O, U1.G
- net E2: now also R4.2; no longer R5.2
- net E2_EN: now also IC2B.O, R3.2; no longer IC1B.O, R2.2
- net E3_EN: now also IC2C.O, R5.2; no longer IC1C.O, R3.2
- net GND: now also IC1.S, IC2D.OE, R5.1; no longer R2.1, U1.S
- net N$1: now also IC1.D, R2.1; no longer R4.1, U1.D
- net N$2: now also R4.1; no longer R5.1
- net PWM: now also IC2A.I, IC2B.I, IC2C.I, IC2D.O; no longer IC1A.I, IC1B.I, IC1C.I, SV1.6
Other:
- moved on the sheet: C1, C2, R2, R3, R4, R5, SV1

Commit message: fixed sch
Parts:
- IC1, IC3, IC4: value DS31126 -> DMN3150L-7
Changed lines of the file:
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@@
 <part name="SUPPLY2" library="supply2" library_urn="urn:adsk.eagle:library:372" deviceset="V+" device=""/>
 <part name="SUPPLY3" library="supply2" library_urn="urn:adsk.eagle:library:372" deviceset="V+" device=""/>
-<part name="IC1" library="ds31126" deviceset="DS31126" device=""/>
-<part name="IC3" library="ds31126" deviceset="DS31126" device=""/>
-<part name="IC4" library="ds31126" deviceset="DS31126" device=""/>
+<part name="IC1" library="ds31126" deviceset="DS31126" device="" value="DMN3150L-7"/>
+<part name="IC3" library="ds31126" deviceset="DS31126" device="" value="DMN3150L-7"/>
+<part name="IC4" library="ds31126" deviceset="DS31126" device="" value="DMN3150L-7"/>
 <part name="GND1" library="supply1" library_urn="urn:adsk.eagle:library:371" deviceset="GND" device=""/>
 <part name="GND2" library="supply1" library_urn="urn:adsk.eagle:library:371" deviceset="GND" device=""/>
@@
 </instance>
 <instance part="IC1" gate="G$1" x="27.94" y="33.02" smashed="yes">
-<attribute name="VALUE" x="16.51" y="33.02" size="1.778" layer="96"/>
-<attribute name="NAME" x="16.51" y="35.56" size="1.778" layer="95"/>
+<attribute name="VALUE" x="11.43" y="33.02" size="1.778" layer="96"/>
+<attribute name="NAME" x="11.43" y="35.56" size="1.778" layer="95"/>
 </instance>
 <instance part="IC3" gate="G$1" x="50.8" y="33.02" smashed="yes">
-<attribute name="VALUE" x="39.37" y="33.02" size="1.778" layer="96"/>
-<attribute name="NAME" x="39.37" y="35.56" size="1.778" layer="95"/>
+<attribute name="VALUE" x="34.29" y="33.02" size="1.778" layer="96"/>
+<attribute name="NAME" x="34.29" y="35.56" size="1.778" layer="95"/>
 </instance>
 <instance part="IC4" gate="G$1" x="73.66" y="33.02" smashed="yes">
-<attribute name="VALUE" x="62.23" y="33.02" size="1.778" layer="96"/>
-<attribute name="NAME" x="62.23" y="35.56" size="1.778" layer="95"/>
+<attribute name="VALUE" x="57.15" y="33.02" size="1.778" layer="96"/>
+<attribute name="NAME" x="57.15" y="35.56" size="1.778" layer="95"/>
 </instance>
 <instance part="GND1" gate="1" x="30.48" y="12.7" smashed="yes">
