File: B-card_rev1/b-card-microcom/rev_001.brd (EAGLE design)
At the start: 160 x 100 mm, 22 parts, among them J1 10118192-0002LF, J2 S2B-PH-SM4-TB(LF)(SN), U1 ATMEGA32U4-MU, U2 MCP73832T-5ACI

Commit message: update
Parts:
- added C6, C7: 10uF, rcl:C0603
- added C9: FC0H104ZFTBR24, FC0H104ZFTBR24:CAPAE1080X580N
- added D1, D2: 10MQ040NTR, diode:DO-214AC
- added L1: 10uH, ul_SDR0403-100ML:IND_BOURNS_SDR0403
- added R7: 100, rcl:R0603
- added U3: TPS61097-33, ul_TPS61097-33DBVR:DBV5-L
- moved C4 155.8 mm to (39.4, 73.7)
- moved C5 155.8 mm to (39.4, 68.6)
- moved LED1 155.8 mm to (39.4, 62.2)
- moved R5 155.8 mm to (39.4, 78.7)
- moved R6 155.8 mm to (39.4, 58.4)
- moved C3 87.2 mm to (50.8, 31.8)
- moved R3 87.2 mm to (50.8, 26.7)
- moved U1 87.2 mm to (53.3, 72.4)
- moved C1 87.2 mm to (50.8, 62.2)
- moved C2 87.2 mm to (50.8, 57.1)
- moved R1 87.2 mm to (50.8, 52.1)
- moved R2 87.2 mm to (50.8, 48.3)
- moved R4 87.2 mm to (50.8, 21.6)
- moved J2 81.1 mm to (15.2, 14.0)
- moved U2 81.1 mm to (24.1, 11.4)
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Connections:
- new net N$10: C6.1, D1.C, D2.C, L1.2, R7.1, U3.1, U3.3
- new net N$8: L1.1, U3.5
- new net N$9: C9.1, D1.A, R7.2
- net +3V3: now also C7.1, U3.4
- net +4.1V: now also D2.A
- net GND: now also C6.2, C7.2, C9.2, U3.2

Commit message: wip
Parts:
- added IC1: DMN2041L-7, ds31126:SOT23
- added NICR1: HOT_WIRE, logo_wire:LAYOUT_A
- added Y1: CSTNE8M00GH5C000R0, CSTNE8M00GH5C000R0:OSC_CSTNE8M00GH5C000R0
Connections:
- new net XTAL1: U1.17, Y1.1
- new net XTAL2: U1.16, Y1.3
- net GND: now also Y1.2
Changed lines of the file:
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@@
 <attribute name="VALUE" x="9.97" y="25.25" size="1.27" layer="27" align="top-left"/>
 </element>
+<element name="Y1" library="CSTNE8M00GH5C000R0" library_urn="urn:adsk.eagle:library:33053036" package="OSC_CSTNE8M00GH5C000R0" package3d_urn="urn:adsk.eagle:package:33053039/1" value="CSTNE8M00GH5C000R0" x="2.54" y="-2.54" smashed="yes">
+<attribute name="DESCRIPTION" value=" 8 MHz Ceramic Resonator Built in Capacitor 33 pF ±0.13% 40 Ohms -40°C ~ 125°C Surface Mount " x="2.54" y="-2.54" size="1.778" layer="27" display="off"/>
+<attribute name="DIGI-KEY_PART_NUMBER" value="490-17961-1-ND" x="2.54" y="-2.54" size="1.778" layer="27" display="off"/>
+<attribute name="MF" value="Murata" x="2.54" y="-2.54" size="1.778" layer="27" display="off"/>
+<attribute name="MP" value="CSTNE8M00GH5C000R0" x="2.54" y="-2.54" size="1.778" layer="27" display="off"/>
+<attribute name="NAME" x="0.54" y="-1.24" size="0.8128" layer="25"/>
+<attribute name="PACKAGE" value="SMD-3 Murata" x="2.54" y="-2.54" size="1.778" layer="27" display="off"/>
+<attribute name="PURCHASE-URL" value="https://pricing.snapeda.com/search/part/CSTNE8M00GH5C000R0/?ref=eda" x="2.54" y="-2.54" size="1.778" layer="27" display="off"/>
+<attribute name="VALUE" x="0.54" y="-3.84" size="0.8128" layer="27" align="top-left"/>
+</element>
+<element name="IC1" library="ds31126" library_urn="urn:adsk.eagle:library:33053132" package="SOT23" package3d_urn="urn:adsk.eagle:package:33053135/1" value="DMN2041L-7" x="2.54" y="-8.89" smashed="yes">
+<attribute name="NAME" x="0.635" y="-6.985" size="1.27" layer="25"/>
+<attribute name="VALUE" x="0.635" y="-12.065" size="1.27" layer="27"/>
+</element>
+<element name="NICR1" library="logo_wire" library_urn="urn:adsk.eagle:library:33053138" package="LAYOUT_A" package3d_urn="urn:adsk.eagle:package:33053143/1" value="HOT_WIRE" x="-3.81" y="12.7" smashed="yes"/>
 </elements>
 <signals>
@@
 <contactref element="C6" pad="2"/>
 <contactref element="C9" pad="2"/>
-<wire x1="32.6" y1="48.26" x2="18.635" y2="31.75" width="0" layer="19" extent="1-1"/>
-<wire x1="32.6" y1="53.34" x2="32.6" y2="48.26" width="0" layer="19" extent="1-1"/>
-<wire x1="31.75635" y1="60.96" x2="32.6" y2="53.34" width="0" layer="19" extent="1-1"/>
-<wire x1="40.22" y1="68.58" x2="31.75635" y2="60.96" width="0" layer="19" extent="1-1"/>
-<wire x1="40.22" y1="73.66" x2="40.22" y2="68.58" width="0" layer="19" extent="1-1"/>
+<contactref element="Y1" pad="2"/>
+<wire x1="53.34" y1="72.39" x2="55.34" y2="75.75" width="0" layer="19" extent="1-1"/>
+<wire x1="49.98" y1="72.89" x2="53.34" y2="72.39" width="0" layer="19" extent="1-1"/>
+<wire x1="51.34" y1="75.75" x2="49.98" y2="72.89" width="0" layer="19" extent="1-1"/>
+<wire x1="52.34" y1="69.03" x2="53.34" y2="72.39" width="0" layer="19" extent="1-1"/>
+<wire x1="56.7" y1="69.89" x2="53.34" y2="72.39" width="0" layer="19" extent="1-1"/>
+<wire x1="51.65" y1="62.23" x2="52.34" y2="69.03" width="0" layer="19" extent="1-1"/>
+<wire x1="51.65" y1="57.15" x2="51.65" y2="62.23" width="0" layer="19" extent="1-1"/>
+<wire x1="40.22" y1="73.66" x2="49.98" y2="72.89" width="0" layer="19" extent="1-1"/>
+<wire x1="40.22" y1="68.58" x2="40.22" y2="73.66" width="0" layer="19" extent="1-1"/>
 <wire x1="38.52" y1="78.74" x2="40.22" y2="73.66" width="0" layer="19" extent="1-1"/>
-<wire x1="16.24" y1="16.9253" x2="38.52" y2="78.74" width="0" layer="19" extent="1-1"/>
+<wire x1="31.75635" y1="60.96" x2="40.22" y2="68.58" width="0" layer="19" extent="1-1"/>
+<wire x1="32.6" y1="53.34" x2="31.75635" y2="60.96" width="0" layer="19" extent="1-1"/>
+<wire x1="32.6" y1="48.26" x2="32.6" y2="53.34" width="0" layer="19" extent="1-1"/>
+<wire x1="39.4" y1="33.02" x2="32.6" y2="48.26" width="0" layer="19" extent="1-1"/>
+<wire x1="51.65" y1="31.75" x2="39.4" y2="33.02" width="0" layer="19" extent="1-1"/>
+<wire x1="49.95" y1="26.67" x2="51.65" y2="31.75" width="0" layer="19" extent="1-1"/>
+<wire x1="18.635" y1="31.75" x2="39.4" y2="33.02" width="0" layer="19" extent="1-1"/>
+<wire x1="16.24" y1="16.9253" x2="18.635" y2="31.75" width="0" layer="19" extent="1-1"/>
 <wire x1="22.8854" y1="11.43" x2="16.24" y2="16.9253" width="0" layer="19" extent="1-1"/>
 <wire x1="35.56" y1="10.16" x2="22.8854" y2="11.43" width="0" layer="19" extent="1-1"/>
-<wire x1="49.95" y1="26.67" x2="35.56" y2="10.16" width="0" layer="19" extent="1-1"/>
-<wire x1="51.65" y1="31.75" x2="49.95" y2="26.67" width="0" layer="19" extent="1-1"/>
-<wire x1="39.4" y1="33.02" x2="51.65" y2="31.75" width="0" layer="19" extent="1-1"/>
-<wire x1="51.65" y1="57.15" x2="39.4" y2="33.02" width="0" layer="19" extent="1-1"/>
-<wire x1="51.65" y1="62.23" x2="51.65" y2="57.15" width="0" layer="19" extent="1-1"/>
-<wire x1="52.34" y1="69.03" x2="51.65" y2="62.23" width="0" layer="19" extent="1-1"/>
-<wire x1="53.34" y1="72.39" x2="52.34" y2="69.03" width="0" layer="19" extent="1-1"/>
-<wire x1="49.98" y1="72.89" x2="53.34" y2="72.39" width="0" layer="19" extent="1-1"/>
-<wire x1="51.34" y1="75.75" x2="49.98" y2="72.89" width="0" layer="19" extent="1-1"/>
-<wire x1="55.34" y1="75.75" x2="53.34" y2="72.39" width="0" layer="19" extent="1-1"/>
-<wire x1="56.7" y1="69.89" x2="53.34" y2="72.39" width="0" layer="19" extent="1-1"/>
+<wire x1="2.54" y1="-2.54" x2="16.24" y2="16.9253" width="0" layer="19" extent="1-1"/>
 </signal>
 <signal name="UVCC">
@@
 <wire x1="27.425" y1="41.91" x2="24.98" y2="25.4" width="0" layer="19" extent="1-1"/>
 </signal>
+<signal name="XTAL1">
+<contactref element="U1" pad="17"/>
+<contactref element="Y1" pad="1"/>
+<wire x1="1.34" y1="-2.54" x2="53.34" y2="69.03" width="0" layer="19" extent="1-1"/>
+</signal>
+<signal name="XTAL2">
+<contactref element="U1" pad="16"/>
+<contactref element="Y1" pad="3"/>
+<wire x1="3.74" y1="-2.54" x2="52.84" y2="69.03" width="0" layer="19" extent="1-1"/>
+</signal>
 </signals>

Commit message: need sleep, 2Bcont
Parts:
- added IC2, IC3: DMN2041L-7, ds31126:SOT23
- added R10, R8, R9: 100k, rcl:R0603
- added SW1: B3AL-1000P, ul_B3AL-1000P:SW_B3AL_OMR
Connections:
- new net E1: IC3.S, NICR1.E1B
- new net E2: IC2.S, NICR1.E2B
- new net E3: IC1.S, NICR1.E3B
- new net N$12: IC1.G, IC2.G, IC3.G, R10.2, R8.2, R9.2
- net +4.1V: now also IC1.D, IC2.D, IC3.D
- net GND: now also NICR1.E1A, NICR1.E2A, NICR1.E3A, R10.1, R8.1, R9.1
Changed lines of the file:
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@@
 </element>
 <element name="NICR1" library="logo_wire" library_urn="urn:adsk.eagle:library:33053138" package="LAYOUT_A" package3d_urn="urn:adsk.eagle:package:33053143/1" value="HOT_WIRE" x="-3.81" y="12.7" smashed="yes"/>
+<element name="R8" library="rcl" library_urn="urn:adsk.eagle:library:334" package="R0603" package3d_urn="urn:adsk.eagle:package:23555/3" value="100k" x="-2.54" y="-15.24" smashed="yes">
+<attribute name="NAME" x="-3.175" y="-14.605" size="1.27" layer="25"/>
+<attribute name="POPULARITY" value="77" x="-2.54" y="-15.24" size="1.778" layer="27" display="off"/>
+<attribute name="SPICEPREFIX" value="R" x="-2.54" y="-15.24" size="1.778" layer="27" display="off"/>
+<attribute name="VALUE" x="-3.175" y="-17.145" size="1.27" layer="27"/>
+</element>
+<element name="IC2" library="ds31126" library_urn="urn:adsk.eagle:library:33053132" package="SOT23" package3d_urn="urn:adsk.eagle:package:33053135/1" value="DMN2041L-7" x="-1.27" y="-21.59" smashed="yes">
+<attribute name="NAME" x="-3.175" y="-19.685" size="1.27" layer="25"/>
+<attribute name="VALUE" x="-3.175" y="-24.765" size="1.27" layer="27"/>
+</element>
+<element name="R9" library="rcl" library_urn="urn:adsk.eagle:library:334" package="R0603" package3d_urn="urn:adsk.eagle:package:23555/3" value="100k" x="-2.54" y="-27.94" smashed="yes">
+<attribute name="NAME" x="-3.175" y="-27.305" size="1.27" layer="25"/>
+<attribute name="POPULARITY" value="77" x="-10.16" y="-20.32" size="1.778" layer="27" display="off"/>
+<attribute name="SPICEPREFIX" value="R" x="-10.16" y="-20.32" size="1.778" layer="27" display="off"/>
+<attribute name="VALUE" x="-3.175" y="-29.845" size="1.27" layer="27"/>
+</element>
+<element name="IC3" library="ds31126" library_urn="urn:adsk.eagle:library:33053132" package="SOT23" package3d_urn="urn:adsk.eagle:package:33053135/1" value="DMN2041L-7" x="-1.27" y="-34.29" smashed="yes">
+<attribute name="NAME" x="-3.175" y="-32.385" size="1.27" layer="25"/>
+<attribute name="VALUE" x="-3.175" y="-37.465" size="1.27" layer="27"/>
+</element>
+<element name="R10" library="rcl" library_urn="urn:adsk.eagle:library:334" package="R0603" package3d_urn="urn:adsk.eagle:package:23555/3" value="100k" x="-2.54" y="-40.64" smashed="yes">
+<attribute name="NAME" x="-3.175" y="-40.005" size="1.27" layer="25"/>
+<attribute name="POPULARITY" value="77" x="-10.16" y="-33.02" size="1.778" layer="27" display="off"/>
+<attribute name="SPICEPREFIX" value="R" x="-10.16" y="-33.02" size="1.778" layer="27" display="off"/>
+<attribute name="VALUE" x="-3.175" y="-42.545" size="1.27" layer="27"/>
+</element>
+<element name="SW1" library="ul_B3AL-1000P" library_urn="urn:adsk.eagle:library:33053187" package="SW_B3AL_OMR" package3d_urn="urn:adsk.eagle:package:33053190/1" value="B3AL-1000P" x="-10.16" y="-36.83" smashed="yes">
+<attribute name="COPYRIGHT" value="Copyright (C) 2021 Ultra Librarian. All rights reserved." x="-10.16" y="-36.83" size="1.778" layer="27" display="off"/>
+<attribute name="DIGI-KEY_PART_NUMBER_1" value="SW1216TR-ND" x="-10.16" y="-36.83" size="1.778" layer="27" display="off"/>
+<attribute name="DIGI-KEY_PART_NUMBER_2" value="SW1216CT-ND" x="-10.16" y="-36.83" size="1.778" layer="27" display="off"/>
+<attribute name="DIGI-KEY_PART_NUMBER_3" value="SW1216DKR-ND" x="-10.16" y="-36.83" size="1.778" layer="27" display="off"/>
+<attribute name="MANUFACTURER_PART_NUMBER" value="B3AL-1000P" x="-10.16" y="-36.83" size="1.778" layer="27" display="off"/>
+<attribute name="MFR_NAME" value="Omron" x="-10.16" y="-36.83" size="1.778" layer="27" display="off"/>
+<attribute name="NAME" x="-12.1666" y="-32.385" size="1.27" layer="27" ratio="6" rot="SR0"/>
+<attribute name="VALUE" x="-11.8872" y="-42.545" size="1.27" layer="21" ratio="6" rot="SR0"/>
+</element>
 </elements>
 <signals>
@@
 <contactref element="C9" pad="2"/>
 <contactref element="Y1" pad="2"/>
+<contactref element="NICR1" pad="E3A"/>
+<contactref element="NICR1" pad="E2A"/>
+<contactref element="NICR1" pad="E1A"/>
+<contactref element="R8" pad="1"/>
+<contactref element="R9" pad="1"/>
+<contactref element="R10" pad="1"/>
 <wire x1="53.34" y1="72.39" x2="55.34" y2="75.75" width="0" layer="19" extent="1-1"/>
 <wire x1="49.98" y1="72.89" x2="53.34" y2="72.39" width="0" layer="19" extent="1-1"/>
@@
 <wire x1="22.8854" y1="11.43" x2="16.24" y2="16.9253" width="0" layer="19" extent="1-1"/>
 <wire x1="35.56" y1="10.16" x2="22.8854" y2="11.43" width="0" layer="19" extent="1-1"/>
-<wire x1="2.54" y1="-2.54" x2="16.24" y2="16.9253" width="0" layer="19" extent="1-1"/>
+<wire x1="-1.31" y1="19.45" x2="16.24" y2="16.9253" width="0" layer="19" extent="1-1"/>
+<wire x1="-3.81" y1="26.45" x2="-1.31" y2="19.45" width="0" layer="19" extent="1-1"/>
+<wire x1="-3.81" y1="12.45" x2="-1.31" y2="19.45" width="0" layer="19" extent="1-1"/>
+<wire x1="2.54" y1="-2.54" x2="-3.81" y2="12.45" width="0" layer="19" extent="1-1"/>
+<wire x1="-3.39" y1="-15.24" x2="2.54" y2="-2.54" width="0" layer="19" extent="1-1"/>
+<wire x1="-3.39" y1="-27.94" x2="-3.39" y2="-15.24" width="0" layer="19" extent="1-1"/>
+<wire x1="-3.39" y1="-40.64" x2="-3.39" y2="-27.94" width="0" layer="19" extent="1-1"/>
 </signal>
 <signal name="UVCC">
@@
 <contactref element="C4" pad="1"/>
 <contactref element="D2" pad="A"/>
-<wire x1="38.52" y1="73.66" x2="27.425" y2="35.56" width="0" layer="19" extent="1-1"/>
-<wire x1="22.8854" y1="10.48" x2="38.52" y2="73.66" width="0" layer="19" extent="1-1"/>
-<wire x1="14.24" y1="16.9253" x2="22.8854" y2="10.48" width="0" layer="19" extent="1-1"/>
+<contactref element="IC1" pad="D"/>
+<contactref element="IC2" pad="D"/>
+<contactref element="IC3" pad="D"/>
+<wire x1="27.425" y1="35.56" x2="38.52" y2="73.66" width="0" layer="19" extent="1-1"/>
+<wire x1="14.24" y1="16.9253" x2="27.425" y2="35.56" width="0" layer="19" extent="1-1"/>
+<wire x1="22.8854" y1="10.48" x2="14.24" y2="16.9253" width="0" layer="19" extent="1-1"/>
+<wire x1="2.54" y1="-7.79" x2="14.24" y2="16.9253" width="0" layer="19" extent="1-1"/>
+<wire x1="-1.27" y1="-20.49" x2="2.54" y2="-7.79" width="0" layer="19" extent="1-1"/>
+<wire x1="-1.27" y1="-33.19" x2="-1.27" y2="-20.49" width="0" layer="19" extent="1-1"/>
 </signal>
 <signal name="N$5">
@@
 <wire x1="3.74" y1="-2.54" x2="52.84" y2="69.03" width="0" layer="19" extent="1-1"/>
 </signal>
+<signal name="E3">
+<contactref element="NICR1" pad="E3B"/>
+<contactref element="IC1" pad="S"/>
+<wire x1="3.49" y1="-9.99" x2="-3.81" y2="-10.55" width="0" layer="19" extent="1-1"/>
+</signal>
+<signal name="E2">
+<contactref element="NICR1" pad="E2B"/>
+<contactref element="IC2" pad="S"/>
+<wire x1="-1.31" y1="9.45" x2="-0.32" y2="-22.69" width="0" layer="19" extent="1-1"/>
+</signal>
+<signal name="E1">
+<contactref element="NICR1" pad="E1B"/>
+<contactref element="IC3" pad="S"/>
+<wire x1="-3.81" y1="16.45" x2="-0.32" y2="-35.39" width="0" layer="19" extent="1-1"/>
+</signal>
+<signal name="N$12">
+<contactref element="IC1" pad="G"/>
+<contactref element="R8" pad="2"/>
+<contactref element="IC2" pad="G"/>
+<contactref element="R9" pad="2"/>
+<contactref element="IC3" pad="G"/>
+<contactref element="R10" pad="2"/>
+<wire x1="-2.22" y1="-35.39" x2="-1.69" y2="-40.64" width="0" layer="19" extent="1-1"/>
+<wire x1="-1.69" y1="-27.94" x2="-2.22" y2="-35.39" width="0" layer="19" extent="1-1"/>
+<wire x1="-2.22" y1="-22.69" x2="-1.69" y2="-27.94" width="0" layer="19" extent="1-1"/>
+<wire x1="-1.69" y1="-15.24" x2="-2.22" y2="-22.69" width="0" layer="19" extent="1-1"/>
+<wire x1="1.59" y1="-9.99" x2="-1.69" y2="-15.24" width="0" layer="19" extent="1-1"/>
+</signal>
 </signals>

Commit message: update
Parts:
- added C10, C11: 1uF, rcl:C0603
- added C8: 0.1uF, rcl:C0603
- added R11: 100k, rcl:R0603
- moved IC2 109.6 mm to (73.7, 58.4)
- moved R10 109.6 mm to (72.4, 39.4)
- moved R8 109.6 mm to (72.4, 64.8)
- moved R9 109.6 mm to (72.4, 52.1)
- moved IC3 109.6 mm to (73.7, 45.7)
- moved SW1 109.6 mm to (64.8, 43.2)
- moved Y1 96.6 mm to (63.5, 72.4)
- moved IC1 79.1 mm to (71.1, 30.5)
- moved NICR1 66.6 mm to (5.08, 78.7)
Connections:
- removed net N$12: IC1.G, IC2.G, IC3.G, R10.2, R8.2, R9.2
- new net D10: IC2.G, R9.2, U1.30
- new net D11: C8.1, R11.1, SW1.2, U1.12
- new net D8: IC3.G, R10.2, U1.28
- new net D9: IC1.G, R8.2, U1.29
- net +3V3: now also C10.1, C11.1, R11.2
- net GND: now also C10.2, C11.2, C8.2, SW1.1

Commit message: update
Parts:
- removed C4, C5: 4.7uF, rcl:C0603
- removed J2: S2B-PH-SM4-TB(LF)(SN), ul_S2B-PH-SM4-TB-LF-SN:CONN_S2B-PH-SM4-TB_JST
- removed R5: 2k, rcl:R0603
- removed U3: TPS61097-33, ul_TPS61097-33DBVR:DBV5-L
- added C14, C15: 470uf, rcl:UD-4X5,8_NICHICON
- added D3: CDBA340-HF, diode:DO-214AC
- added PAD7, PAD8: WIREPAD2,54/0,9, wirepad:2,54/0,9
- added U4: NCP115ASN330T2G, ul_NCP115ASN330T2G:TSOP-5-483-N_ONS
- L1: value 10uH -> 47uh; device ul_SDR0403-100ML:IND_BOURNS_SDR0403 -> Wuerth Elektronik - 7447714470:WUERTH_ELEKTRONIK_7447714470_0
- U2: value MCP73832T-5ACI -> AP1509-50SG-13; device ul_MCP73832T-5ACI-OT:SOT-23-5_MC_MCH-L -> ul_AP1509-50SG-13:SOP-8L_DIO
- moved IC2 70.1 mm to (25.4, 7.62)
- moved U1 67.2 mm to (78.7, 10.2)
- moved C1 62.7 mm to (17.8, 8.89)
- moved L1 56.6 mm to (63.5, 8.89)
- moved U2 56.6 mm to (80.0, 20.3)
- moved R9 53.0 mm to (35.6, 14.0)
- moved R8 51.1 mm to (43.2, 22.9)
- moved NICR1 48.3 mm to (3.81, 30.5)
- moved LED1 44.0 mm to (15.2, 25.4)
- moved C2 39.9 mm to (44.5, 17.8)
- moved R6 36.9 mm to (36.8, 21.6)
- moved Y1 36.1 mm to (52.1, 38.1)
- moved C6 33.0 mm to (30.5, 20.3)
- moved R1 11.7 mm to (43.2, 43.2)
- moved C9 8.98 mm to (15.2, 40.6)
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Connections:
- removed net +4.1V: C4.1, D2.A, IC1.D, IC2.D, IC3.D, J2.1, U2.3
- removed net N$5: R5.2, U2.5
- removed net N$8: L1.1, U3.5
- new net +8V: C14.+, PAD7.1, U2.1
- net +3V3: now also LED1.A, U4.5; no longer U3.4
- net +5V: now also C15.+, D2.A, IC1.D, IC2.D, IC3.D, L1.2, U2.3; no longer C5.1, LED1.A, U2.4
- net GND: now also C14.-, C15.-, D3.A, PAD8.1, R6.1, U2.4, U2.5, U2.6, U2.7, U2.8, U4.2; no longer C4.2, C5.2, J2.2, R5.1, U2.2, U3.2
- net N$10: now also U4.1, U4.3; no longer L1.2, U3.1, U3.3
- net N$7: now also D3.C, L1.1, U2.2; no longer R6.1, U2.1
Other:
- board size 160 x 100 mm -> 88.9 x 50.8 mm
