File: B-card_rev1/b-card-microcom/rev_001.sch (EAGLE design)
At the start: 22 parts, among them J1 10118192-0002LF, J2 S2B-PH-SM4-TB(LF)(SN), U1 ATMEGA32U4-MU, U2 MCP73832T-5ACI

Commit message: update
Parts:
- added C6, C7: 10uF, rcl:C-EUC0603
- added C9: FC0H104ZFTBR24, FC0H104ZFTBR24:FC0H104ZFTBR24
- added D1, D2: 10MQ040NTR, diode:DIODE-DO-214AC
- added L1: 10uH, ul_SDR0403-100ML:IND_BOURNS_SDR0403
- added R7: 100, rcl:R-US_R0603
- added U3: TPS61097-33, ul_TPS61097-33DBVR:TPS61097-33DBVRDBV5-L
Connections:
- new net N$10: C6.1, D1.C, D2.C, L1.2, R7.1, U3.EN, U3.VIN
- new net N$8: L1.1, U3.L
- new net N$9: C9.1, D1.A, R7.2
- net +3V3: now also C7.1, U3.VOUT
- net +4.1V: now also D2.A
- net GND: now also C6.2, C7.2, C9.2, U3.GND
Other:
- note added: "NOTE: still missing xtal"
- note added: "Uber-Cap may blow"
- moved on the sheet: J2

Commit message: wip
Parts:
- added IC1: DMN2041L-7, ds31126:DS31126
- added NICR1: HOT_WIRE, logo_wire:HOT_WIRE
- added Y1: CSTNE8M00GH5C000R0, CSTNE8M00GH5C000R0:CSTNE8M00GH5C000R0
Connections:
- new net XTAL1: U1.XTAL1, Y1.IN
- new net XTAL2: U1.XTAL2, Y1.OUT
- net GND: now also Y1.GND
Other:
- note added: "ALT:TPS61097A-33"
- note added: "Matthew McCardle"
- note removed: "NOTE: still missing xtal"
Changed lines of the file:
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@@
 <part name="SUPPLY3" library="supply2" library_urn="urn:adsk.eagle:library:372" deviceset="+4.1V" device="" value="VBAT"/>
 <part name="C9" library="FC0H104ZFTBR24" library_urn="urn:adsk.eagle:library:33052995" deviceset="FC0H104ZFTBR24" device="" package3d_urn="urn:adsk.eagle:package:33052998/1"/>
+<part name="Y1" library="CSTNE8M00GH5C000R0" library_urn="urn:adsk.eagle:library:33053036" deviceset="CSTNE8M00GH5C000R0" device="" package3d_urn="urn:adsk.eagle:package:33053039/1"/>
+<part name="GND16" library="supply1" library_urn="urn:adsk.eagle:library:371" deviceset="GND" device=""/>
+<part name="IC1" library="ds31126" library_urn="urn:adsk.eagle:library:33053132" deviceset="DS31126" device="" package3d_urn="urn:adsk.eagle:package:33053135/1" value="DMN2041L-7"/>
+<part name="NICR1" library="logo_wire" library_urn="urn:adsk.eagle:library:33053138" deviceset="HOT_WIRE" device="" package3d_urn="urn:adsk.eagle:package:33053143/1"/>
 </parts>
 <sheets>
@@
 <text x="30.48" y="15.24" size="1.27" layer="94">Batt Charger</text>
 <text x="83.82" y="17.78" size="1.27" layer="94" rot="R90">Uber-Cap may blow</text>
-<text x="137.16" y="134.62" size="1.27" layer="94">NOTE: still missing xtal</text>
+<text x="256.54" y="22.86" size="1.6764" layer="94" rot="R180">Matthew McCardle</text>
+<text x="127" y="17.78" size="1.6764" layer="94">ALT:TPS61097A-33</text>
 </plain>
 <instances>
@@
 <attribute name="NAME" x="187.0456" y="53.5686" size="2.0828" layer="95" ratio="6" rot="SR0"/>
 </instance>
-<instance part="GND7" gate="1" x="180.34" y="38.1" smashed="yes">
-<attribute name="VALUE" x="177.8" y="35.56" size="1.778" layer="96"/>
-</instance>
-<instance part="SUPPLY1" gate="P" x="180.34" y="53.34" smashed="yes">
-<attribute name="VALUE" x="178.435" y="56.515" size="1.778" layer="96"/>
+<instance part="GND7" gate="1" x="180.34" y="35.56" smashed="yes">
+<attribute name="VALUE" x="177.8" y="33.02" size="1.778" layer="96"/>
+</instance>
+<instance part="SUPPLY1" gate="P" x="180.34" y="55.88" smashed="yes">
+<attribute name="VALUE" x="178.435" y="59.055" size="1.778" layer="96"/>
 </instance>
 <instance part="R5" gate="G$1" x="60.96" y="25.4" smashed="yes" rot="R90">
@@
 <attribute name="VALUE" x="93.98" y="27.94" size="1.27213125" layer="96" rot="R270"/>
 </instance>
+<instance part="Y1" gate="G$1" x="88.9" y="162.56" smashed="yes">
+<attribute name="NAME" x="81.28" y="168.91" size="1.778" layer="95"/>
+<attribute name="VALUE" x="90.17" y="156.21" size="1.778" layer="96" rot="MR180"/>
+</instance>
+<instance part="GND16" gate="1" x="88.9" y="144.78" smashed="yes">
+<attribute name="VALUE" x="86.36" y="142.24" size="1.778" layer="96"/>
+</instance>
+<instance part="IC1" gate="G$1" x="73.66" y="104.14" smashed="yes">
+<attribute name="VALUE" x="57.15" y="104.14" size="1.778" layer="96"/>
+<attribute name="NAME" x="57.15" y="106.68" size="1.778" layer="95"/>
+</instance>
+<instance part="NICR1" gate="G$1" x="101.6" y="129.54" smashed="yes"/>
+<instance part="NICR1" gate="G$2" x="101.6" y="116.84" smashed="yes"/>
+<instance part="NICR1" gate="G$3" x="101.6" y="104.14" smashed="yes"/>
 </instances>
 <busses>
@@
 <pinref part="J2" gate="A" pin="2"/>
 <wire x1="182.88" y1="45.72" x2="180.34" y2="45.72" width="0.1524" layer="91"/>
-<wire x1="180.34" y1="45.72" x2="180.34" y2="40.64" width="0.1524" layer="91"/>
+<wire x1="180.34" y1="45.72" x2="180.34" y2="38.1" width="0.1524" layer="91"/>
 <pinref part="GND7" gate="1" pin="GND"/>
 </segment>
@@
 <wire x1="88.9" y1="20.32" x2="88.9" y2="17.78" width="0.1524" layer="91"/>
 <pinref part="C9" gate="G$1" pin="2"/>
+</segment>
+<segment>
+<pinref part="Y1" gate="G$1" pin="GND"/>
+<wire x1="88.9" y1="152.4" x2="88.9" y2="147.32" width="0.1524" layer="91"/>
+<pinref part="GND16" gate="1" pin="GND"/>
 </segment>
 </net>
@@
 <pinref part="SUPPLY1" gate="P" pin="+4.1V"/>
 <pinref part="J2" gate="A" pin="1"/>
-<wire x1="180.34" y1="50.8" x2="180.34" y2="48.26" width="0.1524" layer="91"/>
+<wire x1="180.34" y1="53.34" x2="180.34" y2="48.26" width="0.1524" layer="91"/>
 <wire x1="180.34" y1="48.26" x2="182.88" y2="48.26" width="0.1524" layer="91"/>
 </segment>
@@
 </segment>
 </net>
+<net name="XTAL1" class="0">
+<segment>
+<pinref part="U1" gate="G$1" pin="XTAL1"/>
+<wire x1="157.48" y1="137.16" x2="149.86" y2="137.16" width="0.1524" layer="91"/>
+<label x="149.86" y="137.16" size="1.27" layer="95" rot="R180" xref="yes"/>
+</segment>
+<segment>
+<pinref part="Y1" gate="G$1" pin="IN"/>
+<wire x1="76.2" y1="165.1" x2="73.66" y2="165.1" width="0.1524" layer="91"/>
+<label x="73.66" y="165.1" size="1.778" layer="95" rot="R180" xref="yes"/>
+</segment>
+</net>
+<net name="XTAL2" class="0">
+<segment>
+<pinref part="U1" gate="G$1" pin="XTAL2"/>
+<wire x1="157.48" y1="134.62" x2="149.86" y2="134.62" width="0.1524" layer="91"/>
+<label x="149.86" y="134.62" size="1.27" layer="95" rot="R180" xref="yes"/>
+</segment>
+<segment>
+<pinref part="Y1" gate="G$1" pin="OUT"/>
+<wire x1="101.6" y1="165.1" x2="104.14" y2="165.1" width="0.1524" layer="91"/>
+<label x="104.14" y="165.1" size="1.778" layer="95" xref="yes"/>
+</segment>
+</net>

Commit message: need sleep, 2Bcont
Parts:
- added IC2, IC3: DMN2041L-7, ds31126:DS31126
- added R10, R8, R9: 100k, rcl:R-US_R0603
- added SW1: B3AL-1000P, ul_B3AL-1000P:B3AL-1000P
Connections:
- new net E1: IC3.S, NICR1G$1.P$2
- new net E2: IC2.S, NICR1G$2.P$2
- new net E3: IC1.S, NICR1G$3.P$2
- new net N$12: IC1.G, IC2.G, IC3.G, R10.2, R8.2, R9.2
- net +4.1V: now also IC1.D, IC2.D, IC3.D
- net GND: now also NICR1G$1.P$1, NICR1G$2.P$1, NICR1G$3.P$1, R10.1, R8.1, R9.1
Other:
- note added: "Thermal Wire [nickel-chromium]"
- moved on the sheet: IC1, J2, LED1, R6

Commit message: update
Parts:
- added C10, C11: 1uF, rcl:C-EUC0603
- added C8: 0.1uF, rcl:C-EUC0603
- added R11: 100k, rcl:R-US_R0603
Connections:
- removed net N$12: IC1.G, IC2.G, IC3.G, R10.2, R8.2, R9.2
- new net D10: IC2.G, R9.2, U1.PB6(PCINT6/OC1B/OC4B/ADC)
- new net D11: C8.1, R11.1, SW1.2, U1.(PCINT7/OC0A/OC1C/!RTS!)PB7
- new net D8: IC3.G, R10.2, U1.PB4(PCINT4/ADC11)
- new net D9: IC1.G, R8.2, U1.PB5(PCINT5/OC1A/!OC4B!/ADC)
- net +3V3: now also C10.1, C11.1, R11.2
- net GND: now also C10.2, C11.2, C8.2, SW1.1
Other:
- note added: "MCU Ref Design From: Adafruit ItsyBitsy 32u4 - 3V 8MHz"
- note removed: "Ref Design: Adafruit ItsyBitsy 32u4 - 3V 8MHz"
- moved on the sheet: C4, C5, C6, C7, C9, D1, D2, IC1, IC2, IC3, J2, L1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

Commit message: update
Parts:
- removed C4, C5: 4.7uF, rcl:C-EUC0603
- removed J2: S2B-PH-SM4-TB(LF)(SN), ul_S2B-PH-SM4-TB-LF-SN:S2B-PH-SM4-TB(LF)(SN)
- removed R5: 2k, rcl:R-US_R0603
- removed U3: TPS61097-33, ul_TPS61097-33DBVR:TPS61097-33DBVRDBV5-L
- added C14, C15: 470uf, rcl:CPOL-USUD-4X5,8
- added D3: CDBA340-HF, diode:DIODE-DO-214AC
- added PAD7, PAD8: WIREPAD2,54/0,9, wirepad:WIREPAD2,54/0,9
- added U4: NCP115ASN330T2G, ul_NCP115ASN330T2G:NCP115ASN330T2G
- L1: value 10uH -> 47uh; device ul_SDR0403-100ML:IND_BOURNS_SDR0403 -> Wuerth Elektronik - 7447714470:WUERTH_ELEKTRONIK_7447714470WUERTH_ELEKTRONIK_7447714470_0_0
- U2: value MCP73832T-5ACI -> AP1509-50SG-13; device ul_MCP73832T-5ACI-OT:MCP73832T-5ACI/OTSOT-23-5_MC_MCH-L -> ul_AP1509-50SG-13:AP1509-50SG-13
Connections:
- removed net +4.1V: C4.1, D2.A, IC1.D, IC2.D, IC3.D, J2.1, U2.VBAT
- removed net N$5: R5.2, U2.PROG
- removed net N$8: L1.1, U3.L
- new net +8V: C14.+, PAD7.P, U2.VIN
- net +3V3: now also LED1.A, U4.OUT; no longer U3.VOUT
- net +5V: now also C15.+, D2.A, IC1.D, IC2.D, IC3.D, L1.2, U2.FB; no longer C5.1, LED1.A, U2.VDD
- net GND: now also C14.-, C15.-, D3.A, PAD8.P, R6.1, U2.GND, U2.GND_2, U2.GND_3, U2.GND_4, U2.SD, U4.GND; no longer C4.2, C5.2, J2.2, R5.1, U2.VSS, U3.GND
- net N$10: now also U4.EN, U4.IN; no longer L1.2, U3.EN, U3.VIN
- net N$7: now also D3.C, L1.1, U2.OUTPUT; no longer R6.1, U2.STAT
Other:
- note added: "2A limit @ 5vdc"
- note added: "Thermal Business Card"
- note removed: "ALT:TPS61097A-33"
- note removed: "Batt Charger"
- note removed: "Uber-Cap may blow"
- note removed: "VBAT should be fused"
- moved on the sheet: C10, C11, C6, C9, D1, D2, LED1, R6, R7
