File: B-card_rev2/b-card-microcom/rev_002.sch (EAGLE design)
At the start: 47 parts, among them IC1 DMN2041L-7, IC2 DMN2041L-7, IC3 DMN2041L-7, IC4 AZ1117I, IC5 AZ1117I, IC6 AZ1117I, IC7 TLV74033, J1 10118192-0002LF, SW1 B3AL-1000P, U1 ATMEGA32U4-MU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

Commit message: update
this should work, Kinda feel like i should be pushing more current though the elements, but its rev 2, we will see.

Vreg & resistors should stay below the thermal limit. The only thing that should get hot is the activation wire..... mfets should stay cool too i hope.
Parts:
- added C9: 1uF, rcl:C-EUC0603
- D1, D2: value (none) -> LSM115JE3; device diode:DIODE-MINIMELF -> diode:DIODE-DO214BA
- IC4, IC5, IC6: value AZ1117I -> AZ1117IH-5.0
- IC7: value TLV74033 -> AZ1117IH-3.3; device v-reg-micrel:MIC5219XX -> v-reg:LD117ASTR
Connections:
- net +4.1V: now also C9.1; no longer IC7.EN
- net GND: now also C9.2, IC7.ADJ; no longer IC7.GND
Other:
- note added: "1.9 & 0.9 ohms 0.9A & 1.1A"
- note added: "220mv drop | 7.18v & 4.78v"
- note added: "Due to thermal dissipation realworld temp will be < aprox"
- note added: "In open air, E3 will hit 800*c < 60ms E1&E2 will hit 1000*c < 60ms"
- note added: "Should be Fused"
- note added: "The Risk of Fire is real LOL"
- note added: "vreg drop 1.3v | 3.48v 1A = overkill, but only 0.40 cents.."
- note removed: "input voltage > 5.5, vreg will fail, find a better one."
- moved on the sheet: C10, C11, C5, D2, PAD10, PAD9, Y1

Commit message: renum
Parts:
- C1: value 10uF -> 1uF
- C11: value 1uF -> 10uF
- C2, C9: value 1uF -> 0.1uF
- C3, C8: value 0.1uF -> 1uF
- IC1, IC2, IC3: value DMN2041L-7 -> AZ1117IH-5.0; device ds31126:DS31126 -> v-reg:LD117ASTR
- IC4, IC5, IC6: value AZ1117IH-5.0 -> DMN2041L-7; device v-reg:LD117ASTR -> ds31126:DS31126
- PAD1, PAD4: value WIREPADSMD1,27-254 -> WIREPADSMD5-2,5; device wirepad:WIREPADSMD1,27-254 -> wirepad:WIREPADSMD5-2,5
- PAD10, PAD9: value WIREPADSMD5-2,5 -> WIREPADSMD1,27-254; device wirepad:WIREPADSMD5-2,5 -> wirepad:WIREPADSMD1,27-254
- PAD2, PAD3: value WIREPADSMD1,27-254 -> WIREPAD2,54/0,9; device wirepad:WIREPADSMD1,27-254 -> wirepad:WIREPAD2,54/0,9
- PAD7, PAD8: value WIREPAD2,54/0,9 -> WIREPADSMD1,27-254; device wirepad:WIREPAD2,54/0,9 -> wirepad:WIREPADSMD1,27-254
- R1, R2: value 22 -> 11; device rcl:R-US_R0603 -> rcl:R-US_R2512
- R11: value 100k -> 600
- R12, R7: value 11 -> 100k; device rcl:R-US_R2512 -> rcl:R-US_R0603
- R3: value 100k -> 11; device rcl:R-US_R0603 -> rcl:R-US_R2512
- R5: value 11 -> 22; device rcl:R-US_R2512 -> rcl:R-US_R0603
- R6: value 600 -> 22
Connections:
- net !RST: now also PAD6.P, R10.1; no longer PAD1.P, R4.1
- net +3V3: now also C4.1, C6.1, PAD5.P, R10.2, R12.2; no longer C1.1, C10.1, PAD6.P, R11.2, R4.2
- net +4.1V: now also C3.1; no longer C9.1
- net +5V: now also C1.1, IC4.D, IC5.D, IC6.D, R1.2, R2.2, R3.2; no longer C4.1, IC1.D, IC2.D, IC3.D, R12.2, R5.2, R7.2
- net +8V: now also C8.1, IC1.IN, IC2.IN, IC3.IN, PAD1.P, PAD2.P; no longer C6.1, IC4.IN, IC5.IN, IC6.IN, PAD7.P, PAD9.P
- net D+: now also R5.1; no longer R2.1
- net D-: now also R6.1; no longer R1.1
- net D10: now also IC5.G, R8.2; no longer IC2.G, R9.2
- net D11: now also C9.1, R12.1; no longer C8.1, R11.1
- net D8: now also IC4.G, R4.2; no longer IC3.G, R10.2
- net D9: now also IC6.G, R9.2; no longer IC1.G, R8.2
- net E1: now also IC4.S; no longer IC3.S
- net E2: now also IC5.S; no longer IC2.S
- net E3: now also IC6.S; no longer IC1.S
- net GND: now also IC1.ADJ, IC2.ADJ, IC3.ADJ, PAD3.P, PAD4.P, R11.1, R4.1, R7.1; no longer IC4.ADJ, IC5.ADJ, IC6.ADJ, PAD5.P, PAD8.P, R10.1, R3.1, R6.1
- net MISO: now also PAD9.P; no longer PAD4.P
- net MOSI: now also PAD8.P; no longer PAD3.P
- net N$1: now also R6.2; no longer R1.2
- net N$11: now also IC1.OUT, R1.1; no longer IC6.OUT, R12.1
- net N$2: now also C10.1; no longer C2.1
- net N$3: now also R5.2; no longer R2.2
- net N$4: now also C2.1, R7.2; no longer C3.1, R3.2
- net N$6: now also R11.2; no longer R6.2
- net N$7: now also IC3.OUT, R3.1; no longer IC4.OUT, R7.1
- net N$9: now also IC2.OUT, R2.1; no longer IC5.OUT, R5.1
- net SCK: now also PAD7.P; no longer PAD2.P
Other:
- note added: "Dont Strobe E1+E2+E3, only one at a time."
- note added: "No ETA on battery life"
- moved on the sheet: C1, C10, C11, C2, C3, C4, C6, C7, C8, C9, PAD1, PAD10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

Commit message: layout kinda done
I'm not 100% happy with everything yet, but it looks like it could work.
Parts:
- added C12, C13, C14, C15, C16: 1uF, rcl:C-EUC0603
Connections:
- net D+ renamed USBA_P
- net D- renamed USBA_N
- net N$1 renamed USBB_N
- net N$3 renamed USBB_P
- removed net D11: C9.1, R12.1, SW1.2, U1.(PCINT7/OC0A/OC1C/!RTS!)PB7
- new net D6: IC4.G, R4.2, U1.PD7(T0/OC4D/ADC10)
- new net VBUS: D1.A, J1.VCC, U1.VBUS
- net +3V3: now also C14.1, C15.1, C16.1
- net +5V: now also C12.1, C13.1; no longer D1.A, J1.VCC, U1.VBUS
- net D10: now also C9.1, R12.1, SW1.2; no longer IC5.G, R8.2
- net D8: now also IC5.G, R8.2; no longer IC4.G, R4.2
- net GND: now also C12.2, C13.2, C14.2, C15.2, C16.2
Other:
- moved on the sheet: C4, C6, Y1

Commit message: update
Parts:
- C14, C15, C16, C4, C6: value 1uF -> 0.1uF
Other:
- note added: "https://www.digikey.com/short/cp92bq0z"
Changed lines of the file:
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@@
 <part name="+3V6" library="supply1" library_urn="urn:adsk.eagle:library:371" deviceset="+3V3" device=""/>
 <part name="GND22" library="supply1" library_urn="urn:adsk.eagle:library:371" deviceset="GND" device=""/>
-<part name="C4" library="rcl" library_urn="urn:adsk.eagle:library:334" deviceset="C-EU" device="C0603" package3d_urn="urn:adsk.eagle:package:23616/2" value="1uF"/>
-<part name="C6" library="rcl" library_urn="urn:adsk.eagle:library:334" deviceset="C-EU" device="C0603" package3d_urn="urn:adsk.eagle:package:23616/2" value="1uF"/>
+<part name="C4" library="rcl" library_urn="urn:adsk.eagle:library:334" deviceset="C-EU" device="C0603" package3d_urn="urn:adsk.eagle:package:23616/2" value="0.1uF"/>
+<part name="C6" library="rcl" library_urn="urn:adsk.eagle:library:334" deviceset="C-EU" device="C0603" package3d_urn="urn:adsk.eagle:package:23616/2" value="0.1uF"/>
 <part name="GND23" library="supply1" library_urn="urn:adsk.eagle:library:371" deviceset="GND" device=""/>
 <part name="GND24" library="supply1" library_urn="urn:adsk.eagle:library:371" deviceset="GND" device=""/>
@@
 <part name="GND14" library="supply1" library_urn="urn:adsk.eagle:library:371" deviceset="GND" device=""/>
 <part name="GND15" library="supply1" library_urn="urn:adsk.eagle:library:371" deviceset="GND" device=""/>
-<part name="C14" library="rcl" library_urn="urn:adsk.eagle:library:334" deviceset="C-EU" device="C0603" package3d_urn="urn:adsk.eagle:package:23616/2" value="1uF"/>
-<part name="C15" library="rcl" library_urn="urn:adsk.eagle:library:334" deviceset="C-EU" device="C0603" package3d_urn="urn:adsk.eagle:package:23616/2" value="1uF"/>
+<part name="C14" library="rcl" library_urn="urn:adsk.eagle:library:334" deviceset="C-EU" device="C0603" package3d_urn="urn:adsk.eagle:package:23616/2" value="0.1uF"/>
+<part name="C15" library="rcl" library_urn="urn:adsk.eagle:library:334" deviceset="C-EU" device="C0603" package3d_urn="urn:adsk.eagle:package:23616/2" value="0.1uF"/>
 <part name="+3V10" library="supply1" library_urn="urn:adsk.eagle:library:371" deviceset="+3V3" device=""/>
 <part name="+3V11" library="supply1" library_urn="urn:adsk.eagle:library:371" deviceset="+3V3" device=""/>
 <part name="GND26" library="supply1" library_urn="urn:adsk.eagle:library:371" deviceset="GND" device=""/>
 <part name="GND27" library="supply1" library_urn="urn:adsk.eagle:library:371" deviceset="GND" device=""/>
-<part name="C16" library="rcl" library_urn="urn:adsk.eagle:library:334" deviceset="C-EU" device="C0603" package3d_urn="urn:adsk.eagle:package:23616/2" value="1uF"/>
+<part name="C16" library="rcl" library_urn="urn:adsk.eagle:library:334" deviceset="C-EU" device="C0603" package3d_urn="urn:adsk.eagle:package:23616/2" value="0.1uF"/>
 <part name="GND28" library="supply1" library_urn="urn:adsk.eagle:library:371" deviceset="GND" device=""/>
 <part name="+3V12" library="supply1" library_urn="urn:adsk.eagle:library:371" deviceset="+3V3" device=""/>
@@
 E1&amp;E2 will hit 1000*c &lt; 60ms</text>
 <text x="38.1" y="50.8" size="1.778" layer="94">Due to thermal dissipation realworld temp will be &lt; aprox</text>
-<text x="172.72" y="12.7" size="1.778" layer="94">The Risk of Fire is real LOL</text>
+<text x="172.72" y="15.24" size="1.778" layer="94">The Risk of Fire is real LOL</text>
 <text x="170.18" y="160.02" size="1.778" layer="94">Dont Strobe E1+E2+E3, only one at a time.</text>
 <text x="132.08" y="53.34" size="1.778" layer="94">No ETA on battery life</text>
+<text x="165.1" y="10.16" size="1.778" layer="94">https://www.digikey.com/short/cp92bq0z</text>
 </plain>
 <instances>
@@
 </instance>
 <instance part="R10" gate="G$1" x="154.94" y="152.4" smashed="yes" rot="R90">
-<attribute name="NAME" x="158.5214" y="148.59" size="1.778" layer="95" rot="R90"/>
-<attribute name="VALUE" x="158.242" y="153.67" size="1.778" layer="96" rot="R90"/>
+<attribute name="NAME" x="153.4414" y="151.13" size="1.778" layer="95" rot="R90"/>
+<attribute name="VALUE" x="158.242" y="151.13" size="1.778" layer="96" rot="R90"/>
 </instance>
 <instance part="+3V3" gate="G$1" x="154.94" y="165.1" smashed="yes">
@@
 </instance>
 <instance part="R11" gate="G$1" x="182.88" y="43.18" smashed="yes" rot="R90">
-<attribute name="NAME" x="186.4614" y="39.37" size="1.778" layer="95" rot="R90"/>
-<attribute name="VALUE" x="186.182" y="44.45" size="1.778" layer="96" rot="R90"/>
+<attribute name="NAME" x="181.3814" y="41.91" size="1.778" layer="95" rot="R90"/>
+<attribute name="VALUE" x="186.182" y="41.91" size="1.778" layer="96" rot="R90"/>
 </instance>
 <instance part="Y1" gate="G$1" x="134.62" y="83.82" smashed="yes">
@@
 </instance>
 <instance part="R9" gate="G$1" x="104.14" y="20.32" smashed="yes" rot="R90">
-<attribute name="NAME" x="107.7214" y="16.51" size="1.778" layer="95" rot="R90"/>
-<attribute name="VALUE" x="107.442" y="21.59" size="1.778" layer="96" rot="R90"/>
+<attribute name="NAME" x="102.6414" y="19.05" size="1.778" layer="95" rot="R90"/>
+<attribute name="VALUE" x="107.442" y="19.05" size="1.778" layer="96" rot="R90"/>
 </instance>
 <instance part="GND18" gate="1" x="104.14" y="10.16" smashed="yes">
@@
 </instance>
 <instance part="R8" gate="G$1" x="76.2" y="20.32" smashed="yes" rot="R90">
-<attribute name="NAME" x="79.7814" y="16.51" size="1.778" layer="95" rot="R90"/>
-<attribute name="VALUE" x="79.502" y="21.59" size="1.778" layer="96" rot="R90"/>
+<attribute name="NAME" x="74.7014" y="19.05" size="1.778" layer="95" rot="R90"/>
+<attribute name="VALUE" x="79.502" y="19.05" size="1.778" layer="96" rot="R90"/>
 </instance>
 <instance part="GND19" gate="1" x="76.2" y="10.16" smashed="yes">
@@
 </instance>
 <instance part="R4" gate="G$1" x="48.26" y="20.32" smashed="yes" rot="R90">
-<attribute name="NAME" x="51.8414" y="13.97" size="1.778" layer="95" rot="R90"/>
-<attribute name="VALUE" x="51.562" y="21.59" size="1.778" layer="96" rot="R90"/>
+<attribute name="NAME" x="46.7614" y="19.05" size="1.778" layer="95" rot="R90"/>
+<attribute name="VALUE" x="51.562" y="19.05" size="1.778" layer="96" rot="R90"/>
 </instance>
 <instance part="GND20" gate="1" x="48.26" y="10.16" smashed="yes">
@@
 </instance>
 <instance part="R12" gate="G$1" x="205.74" y="60.96" smashed="yes" rot="R90">
-<attribute name="NAME" x="209.3214" y="54.61" size="1.778" layer="95" rot="R90"/>
-<attribute name="VALUE" x="209.042" y="62.23" size="1.778" layer="96" rot="R90"/>
+<attribute name="NAME" x="204.2414" y="59.69" size="1.778" layer="95" rot="R90"/>
+<attribute name="VALUE" x="209.042" y="59.69" size="1.778" layer="96" rot="R90"/>
 </instance>
 <instance part="GND21" gate="1" x="205.74" y="30.48" smashed="yes">

Commit message: updated
Parts:
- IC1, IC2, IC3, IC7: device v-reg:LD117ASTR -> v-reg-edit:AZ1117IH
- LED1: device led:LEDSML0603 -> led_edit:LEDSML0603
Changed lines of the file:
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@@
 <parts>
 <part name="FRAME1" library="frames" library_urn="urn:adsk.eagle:library:229" deviceset="A4L-LOC" device=""/>
-<part name="U1" library="ATMEGA32U4-MU" library_urn="urn:adsk.eagle:library:33052628" deviceset="ATMEGA32U4-MU" device="" package3d_urn="urn:adsk.eagle:package:33052631/1"/>
+<part name="U1" library="ATMEGA32U4-MU" library_urn="urn:adsk.eagle:library:33052628" deviceset="ATMEGA32U4-MU" device="" package3d_urn="urn:adsk.eagle:package:33052631/2"/>
 <part name="+3V1" library="supply1" library_urn="urn:adsk.eagle:library:371" deviceset="+3V3" device=""/>
 <part name="GND1" library="supply1" library_urn="urn:adsk.eagle:library:371" deviceset="GND" device=""/>
@@
 <part name="R6" library="rcl" library_urn="urn:adsk.eagle:library:334" deviceset="R-US_" device="R0603" package3d_urn="urn:adsk.eagle:package:23555/3" value="22"/>
 <part name="R5" library="rcl" library_urn="urn:adsk.eagle:library:334" deviceset="R-US_" device="R0603" package3d_urn="urn:adsk.eagle:package:23555/3" value="22"/>
-<part name="J1" library="10118192-0002LF" library_urn="urn:adsk.eagle:library:33052679" deviceset="10118192-0002LF" device="" package3d_urn="urn:adsk.eagle:package:33052682/1"/>
+<part name="J1" library="10118192-0002LF" library_urn="urn:adsk.eagle:library:33052679" deviceset="10118192-0002LF" device="" package3d_urn="urn:adsk.eagle:package:33052682/2"/>
 <part name="GND4" library="supply1" library_urn="urn:adsk.eagle:library:371" deviceset="GND" device=""/>
 <part name="C2" library="rcl" library_urn="urn:adsk.eagle:library:334" deviceset="C-EU" device="C0603" package3d_urn="urn:adsk.eagle:package:23616/2" value="0.1uF"/>
@@
 <part name="+3V4" library="supply1" library_urn="urn:adsk.eagle:library:371" deviceset="+3V3" device=""/>
 <part name="GND6" library="supply1" library_urn="urn:adsk.eagle:library:371" deviceset="GND" device=""/>
-<part name="LED1" library="led" library_urn="urn:adsk.eagle:library:259" deviceset="LED" device="SML0603" package3d_urn="urn:adsk.eagle:package:15832/1"/>
+<part name="LED1" library="led_edit" library_urn="urn:adsk.eagle:library:33236245" deviceset="LED" device="SML0603" package3d_urn="urn:adsk.eagle:package:33236243/2"/>
 <part name="R11" library="rcl" library_urn="urn:adsk.eagle:library:334" deviceset="R-US_" device="R0603" package3d_urn="urn:adsk.eagle:package:23555/3" value="600"/>
-<part name="Y1" library="CSTNE8M00GH5C000R0" library_urn="urn:adsk.eagle:library:33053036" deviceset="CSTNE8M00GH5C000R0" device="" package3d_urn="urn:adsk.eagle:package:33053039/1"/>
+<part name="Y1" library="CSTNE8M00GH5C000R0" library_urn="urn:adsk.eagle:library:33053036" deviceset="CSTNE8M00GH5C000R0" device="" package3d_urn="urn:adsk.eagle:package:33053039/2"/>
 <part name="GND16" library="supply1" library_urn="urn:adsk.eagle:library:371" deviceset="GND" device=""/>
-<part name="IC6" library="ds31126" library_urn="urn:adsk.eagle:library:33053132" deviceset="DS31126" device="" package3d_urn="urn:adsk.eagle:package:33053135/1" value="DMN2041L-7"/>
+<part name="IC6" library="ds31126" library_urn="urn:adsk.eagle:library:33053132" deviceset="DS31126" device="" package3d_urn="urn:adsk.eagle:package:33053135/3" value="DMN2041L-7"/>
 <part name="NICR1" library="logo_wire" library_urn="urn:adsk.eagle:library:33053138" deviceset="HOT_WIRE" device="" package3d_urn="urn:adsk.eagle:package:33053143/1"/>
 <part name="GND17" library="supply1" library_urn="urn:adsk.eagle:library:371" deviceset="GND" device=""/>
 <part name="R9" library="rcl" library_urn="urn:adsk.eagle:library:334" deviceset="R-US_" device="R0603" package3d_urn="urn:adsk.eagle:package:23555/3" value="100k"/>
 <part name="GND18" library="supply1" library_urn="urn:adsk.eagle:library:371" deviceset="GND" device=""/>
-<part name="IC5" library="ds31126" library_urn="urn:adsk.eagle:library:33053132" deviceset="DS31126" device="" package3d_urn="urn:adsk.eagle:package:33053135/1" value="DMN2041L-7"/>
+<part name="IC5" library="ds31126" library_urn="urn:adsk.eagle:library:33053132" deviceset="DS31126" device="" package3d_urn="urn:adsk.eagle:package:33053135/3" value="DMN2041L-7"/>
 <part name="R8" library="rcl" library_urn="urn:adsk.eagle:library:334" deviceset="R-US_" device="R0603" package3d_urn="urn:adsk.eagle:package:23555/3" value="100k"/>
 <part name="GND19" library="supply1" library_urn="urn:adsk.eagle:library:371" deviceset="GND" device=""/>
-<part name="IC4" library="ds31126" library_urn="urn:adsk.eagle:library:33053132" deviceset="DS31126" device="" package3d_urn="urn:adsk.eagle:package:33053135/1" value="DMN2041L-7"/>
+<part name="IC4" library="ds31126" library_urn="urn:adsk.eagle:library:33053132" deviceset="DS31126" device="" package3d_urn="urn:adsk.eagle:package:33053135/3" value="DMN2041L-7"/>
 <part name="R4" library="rcl" library_urn="urn:adsk.eagle:library:334" deviceset="R-US_" device="R0603" package3d_urn="urn:adsk.eagle:package:23555/3" value="100k"/>
 <part name="GND20" library="supply1" library_urn="urn:adsk.eagle:library:371" deviceset="GND" device=""/>
-<part name="SW1" library="ul_B3AL-1000P" library_urn="urn:adsk.eagle:library:33053187" deviceset="B3AL-1000P" device="" package3d_urn="urn:adsk.eagle:package:33053190/2"/>
+<part name="SW1" library="ul_B3AL-1000P" library_urn="urn:adsk.eagle:library:33053187" deviceset="B3AL-1000P" device="" package3d_urn="urn:adsk.eagle:package:33053190/3"/>
 <part name="C9" library="rcl" library_urn="urn:adsk.eagle:library:334" deviceset="C-EU" device="C0603" package3d_urn="urn:adsk.eagle:package:23616/2" value="0.1uF"/>
 <part name="R12" library="rcl" library_urn="urn:adsk.eagle:library:334" deviceset="R-US_" device="R0603" package3d_urn="urn:adsk.eagle:package:23555/3" value="100k"/>
@@
 <part name="SUPPLY8" library="supply2" library_urn="urn:adsk.eagle:library:372" deviceset="+8V" device="" value="VBAT"/>
 <part name="GND30" library="supply1" library_urn="urn:adsk.eagle:library:371" deviceset="GND" device=""/>
-<part name="IC3" library="v-reg" library_urn="urn:adsk.eagle:library:409" deviceset="LD117A?*" device="S" package3d_urn="urn:adsk.eagle:package:30370/1" technology="TR" value="AZ1117IH-5.0"/>
+<part name="IC3" library="v-reg-edit" library_urn="urn:adsk.eagle:library:33236191" deviceset="AZ1117IH" device="" package3d_urn="urn:adsk.eagle:package:33236198/2" value="AZ1117IH-5.0"/>
 <part name="GND7" library="supply1" library_urn="urn:adsk.eagle:library:371" deviceset="GND" device=""/>
 <part name="R3" library="rcl" library_urn="urn:adsk.eagle:library:334" deviceset="R-US_" device="R2512" package3d_urn="urn:adsk.eagle:package:23545/2" value="11"/>
-<part name="IC2" library="v-reg" library_urn="urn:adsk.eagle:library:409" deviceset="LD117A?*" device="S" package3d_urn="urn:adsk.eagle:package:30370/1" technology="TR" value="AZ1117IH-5.0"/>
+<part name="IC2" library="v-reg-edit" library_urn="urn:adsk.eagle:library:33236191" deviceset="AZ1117IH" device="" package3d_urn="urn:adsk.eagle:package:33236198/2" value="AZ1117IH-5.0"/>
 <part name="GND8" library="supply1" library_urn="urn:adsk.eagle:library:371" deviceset="GND" device=""/>
 <part name="R2" library="rcl" library_urn="urn:adsk.eagle:library:334" deviceset="R-US_" device="R2512" package3d_urn="urn:adsk.eagle:package:23545/2" value="11"/>
-<part name="IC1" library="v-reg" library_urn="urn:adsk.eagle:library:409" deviceset="LD117A?*" device="S" package3d_urn="urn:adsk.eagle:package:30370/1" technology="TR" value="AZ1117IH-5.0"/>
+<part name="IC1" library="v-reg-edit" library_urn="urn:adsk.eagle:library:33236191" deviceset="AZ1117IH" device="" package3d_urn="urn:adsk.eagle:package:33236198/2" value="AZ1117IH-5.0"/>
 <part name="GND9" library="supply1" library_urn="urn:adsk.eagle:library:371" deviceset="GND" device=""/>
 <part name="R1" library="rcl" library_urn="urn:adsk.eagle:library:334" deviceset="R-US_" device="R2512" package3d_urn="urn:adsk.eagle:package:23545/2" value="11"/>
@@
 <part name="PAD1" library="wirepad" library_urn="urn:adsk.eagle:library:412" deviceset="WIREPAD" device="SMD5-2,5" package3d_urn="urn:adsk.eagle:package:30845/1"/>
 <part name="PAD4" library="wirepad" library_urn="urn:adsk.eagle:library:412" deviceset="WIREPAD" device="SMD5-2,5" package3d_urn="urn:adsk.eagle:package:30845/1"/>
-<part name="IC7" library="v-reg" library_urn="urn:adsk.eagle:library:409" deviceset="LD117A?*" device="S" package3d_urn="urn:adsk.eagle:package:30370/1" technology="TR" value="AZ1117IH-3.3"/>
+<part name="IC7" library="v-reg-edit" library_urn="urn:adsk.eagle:library:33236191" deviceset="AZ1117IH" device="" package3d_urn="urn:adsk.eagle:package:33236198/2" value="AZ1117IH-3.3"/>
 <part name="C3" library="rcl" library_urn="urn:adsk.eagle:library:334" deviceset="C-EU" device="C0603" package3d_urn="urn:adsk.eagle:package:23616/2" value="1uF"/>
 <part name="GND13" library="supply1" library_urn="urn:adsk.eagle:library:371" deviceset="GND" device=""/>

Commit message: update
Connections:
- net USBA_N: now also R5.1; no longer R6.1
- net USBA_P: now also R6.1; no longer R5.1
- net USBB_N: now also J1.D-, R5.2; no longer J1.D+, R6.2
- net USBB_P: now also J1.D+, R6.2; no longer J1.D-, R5.2
Changed lines of the file:
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@@
 </segment>
 </net>
-<net name="USBB_N" class="0">
+<net name="USBB_P" class="0">
 <segment>
 <pinref part="J1" gate="G$1" pin="D+"/>
@@
 </segment>
 </net>
-<net name="USBB_P" class="0">
+<net name="USBB_N" class="0">
 <segment>
 <pinref part="J1" gate="G$1" pin="D-"/>
@@
 </segment>
 <segment>
+<pinref part="R6" gate="G$1" pin="1"/>
+<wire x1="55.88" y1="154.94" x2="53.34" y2="154.94" width="0.1524" layer="91"/>
+<label x="53.34" y="154.94" size="1.27" layer="95" rot="R180" xref="yes"/>
+</segment>
+</net>
+<net name="USBA_N" class="0">
+<segment>
+<pinref part="U1" gate="G$1" pin="D-"/>
+<wire x1="228.6" y1="137.16" x2="231.14" y2="137.16" width="0.1524" layer="91"/>
+<label x="231.14" y="137.16" size="1.27" layer="95" xref="yes"/>
+</segment>
+<segment>
 <pinref part="R5" gate="G$1" pin="1"/>
 <wire x1="55.88" y1="160.02" x2="53.34" y2="160.02" width="0.1524" layer="91"/>
@@
 </segment>
 </net>
-<net name="USBA_N" class="0">
-<segment>
-<pinref part="U1" gate="G$1" pin="D-"/>
-<wire x1="228.6" y1="137.16" x2="231.14" y2="137.16" width="0.1524" layer="91"/>
-<label x="231.14" y="137.16" size="1.27" layer="95" xref="yes"/>
-</segment>
-<segment>
-<pinref part="R6" gate="G$1" pin="1"/>
-<wire x1="55.88" y1="154.94" x2="53.34" y2="154.94" width="0.1524" layer="91"/>
-<label x="53.34" y="154.94" size="1.27" layer="95" rot="R180" xref="yes"/>
-</segment>
-</net>
